File: panels_controller_nano.sch (KiCad schematic (older format))
At the start: 10 parts, among them J1 DB9, K1 PB5, K2 PE6

Commit message: Modified nano in lib file
Parts:
- removed D1: LED, symbol LED
- removed R3: 300, symbol R
Connections:
- wire segments 37 -> 18
Other:
- moved on the sheet: J1, K1, K2, R1, R2, U?

Commit message: Completed Ver. 1.0 board design.
Parts:
- removed C2: 0.1uF, symbol C
- added C2: 10uF, symbol CAPAPOL
- added C3: 0.33uF, symbol C
- added P1: CONN_2X2, symbol CONN_2X2
- added P2, P3, P4, P5: CONN_1, symbol CONN_1
- added R3: 68, symbol R
- C1: value 10uF -> 0.1uF
- J1: value DB9 -> DB9_FEMALE_PINS
- K1: value PB5 -> PD3
- K2: value PE6 -> PB1
- gave numbers to parts that had none: 1
Connections:
- net labels added: PB1, PD3, RST, SCL, SDA
- wire segments 18 -> 52
- no-connect marks 6 -> 29
Other:
- moved on the sheet: J1, K1, K2, R1, R2, U1

Commit message: Board version 2.0
Parts:
- removed C1: 0.1uF, symbol C
- removed C2: 10uF, symbol CAPAPOL
- removed C3: 0.33uF, symbol C
- removed P1: CONN_2X2, symbol CONN_2X2
- removed R3: 68, symbol R
Connections:
- net labels removed: RST
- wire segments 52 -> 38
Changed lines of the file:
@@
-EESchema Schematic File Version 2  date Tue 08 Feb 2011 02:38:41 PM PST
+EESchema Schematic File Version 2  date Wed 16 Feb 2011 03:37:27 PM PST
 LIBS:power
 LIBS:device
@@
 Sheet 1 1
 Title "panels_controller_nano"
-Date "8 feb 2011"
-Rev "1.0"
+Date "16 feb 2011"
+Rev "2.0"
 Comp ""
 Comment1 ""
@@
 Comment4 ""
 $EndDescr
+Connection ~ 3950 4850
+Wire Wire Line
+	4200 5200 3950 5200
+Wire Wire Line
+	3950 5200 3950 4850
 Connection ~ 6150 6000
 Wire Wire Line
-	6250 6000 6150 6000
+	6150 6000 6250 6000
 Connection ~ 6150 5700
 Wire Wire Line
 	6250 5700 6150 5700
 Wire Wire Line
-	8050 5750 8050 5900
-Connection ~ 8050 5250
-Wire Wire Line
-	7700 5250 8050 5250
-Connection ~ 8050 4950
-Wire Wire Line
-	7850 4950 8050 4950
-Wire Wire Line
-	7050 4850 6750 4850
-Connection ~ 5400 5400
-Wire Wire Line
-	5800 5400 5000 5400
-Connection ~ 5200 5400
-Wire Wire Line
-	5200 5400 5200 5600
-Wire Wire Line
-	5400 4900 5400 4950
-Wire Wire Line
-	5000 4950 5000 4900
-Wire Wire Line
 	6350 2700 6350 2650
 Wire Wire Line
@@
 	4100 4750 3350 4750
 Wire Wire Line
-	6000 2750 6250 2750
-Wire Wire Line
 	4300 2850 4150 2850
 Wire Wire Line
@@
 Wire Wire Line
 	6350 3000 6350 2900
-Wire Wire Line
-	5000 5400 5000 5350
-Wire Wire Line
-	5400 5400 5400 5350
-Wire Wire Line
-	5200 4900 5200 4700
-Connection ~ 5200 4900
-Wire Wire Line
-	5000 4900 5800 4900
-Connection ~ 5400 4900
-Wire Wire Line
-	7850 4850 8050 4850
-Wire Wire Line
-	8050 4850 8050 5350
-Wire Wire Line
-	7200 5250 6750 5250
-Wire Wire Line
-	6750 5250 6750 5150
 Wire Wire Line
 	6250 5550 6150 5550
@@
 	6250 5850 6150 5850
 Connection ~ 6150 5850
-$Comp
-L GND #PWR15
+Wire Wire Line
+	4000 4350 4000 4650
+Connection ~ 4000 4650
+$Comp
+L PWR_FLAG #FLG01
+U 1 1 4D5C5F9C
+P 4200 5200
+F 0 "#FLG01" H 4200 5470 30  0001 C CNN
+F 1 "PWR_FLAG" H 4200 5430 30  0000 C CNN
+	1    4200 5200
+	1    0    0    -1
+$EndComp
+$Comp
+L PWR_FLAG #FLG02
+U 1 1 4D5C5F88
+P 4000 4350
+F 0 "#FLG02" H 4000 4620 30  0001 C CNN
+F 1 "PWR_FLAG" H 4000 4580 30  0000 C CNN
+	1    4000 4350
+	1    0    0    -1
+$EndComp
+NoConn ~ 6000 2750
+$Comp
+L GND #PWR03
 U 1 1 4D51C5D1
 P 6150 6200
-F 0 "#PWR15" H 6150 6200 30  0001 C CNN
+F 0 "#PWR03" H 6150 6200 30  0001 C CNN
 F 1 "GND" H 6150 6130 30  0001 C CNN
 	1    6150 6200
@@
 $EndComp
 $Comp
-L GND #PWR14
-U 1 1 4D51BA9B
-P 8050 5900
-F 0 "#PWR14" H 8050 5900 30  0001 C CNN
-F 1 "GND" H 8050 5830 30  0001 C CNN
-	1    8050 5900
-	1    0    0    -1
-$EndComp
-$Comp
-L +5V #PWR10
-U 1 1 4D51BA90
-P 6750 5150
-F 0 "#PWR10" H 6750 5240 20  0001 C CNN
-F 1 "+5V" H 6750 5240 30  0000 C CNN
-	1    6750 5150
-	1    0    0    -1
-$EndComp
-$Comp
-L R R3
-U 1 1 4D51BA3D
-P 7450 5250
-F 0 "R3" V 7530 5250 50  0000 C CNN
-F 1 "68" V 7450 5250 50  0000 C CNN
-	1    7450 5250
-	0    1    1    0
-$EndComp
-$Comp
-L C C3
-U 1 1 4D51BA2F
-P 8050 5550
-F 0 "C3" H 8100 5650 50  0000 L CNN
-F 1 "0.33uF" H 8100 5450 50  0000 L CNN
-	1    8050 5550
-	1    0    0    -1
-$EndComp
-Text Label 6800 4850 0    60   ~ 0
-RST
-NoConn ~ 7050 4950
-$Comp
-L CONN_2X2 P1
-U 1 1 4D51B9CC
-P 7450 4900
-F 0 "P1" H 7450 5050 50  0000 C CNN
-F 1 "CONN_2X2" H 7460 4770 40  0000 C CNN
-	1    7450 4900
-	1    0    0    -1
-$EndComp
-$Comp
-L PWR_FLAG #FLG2
-U 1 1 4D51B947
-P 5800 5400
-F 0 "#FLG2" H 5800 5670 30  0001 C CNN
-F 1 "PWR_FLAG" H 5800 5630 30  0000 C CNN
-	1    5800 5400
-	1    0    0    -1
-$EndComp
-$Comp
-L PWR_FLAG #FLG1
-U 1 1 4D51B941
-P 5800 4900
-F 0 "#FLG1" H 5800 5170 30  0001 C CNN
-F 1 "PWR_FLAG" H 5800 5130 30  0000 C CNN
-	1    5800 4900
-	1    0    0    -1
-$EndComp
-$Comp
-L CAPAPOL C2
-U 1 1 4D51B8F1
-P 5400 5150
-F 0 "C2" H 5450 5250 50  0000 L CNN
-F 1 "10uF" H 5450 5050 50  0000 L CNN
-	1    5400 5150
-	1    0    0    -1
-$EndComp
-$Comp
-L C C1
-U 1 1 4D51B8E7
-P 5000 5150
-F 0 "C1" H 5050 5250 50  0000 L CNN
-F 1 "0.1uF" H 5050 5050 50  0000 L CNN
-	1    5000 5150
-	1    0    0    -1
-$EndComp
-Text Label 6050 2750 0    60   ~ 0
-RST
-$Comp
-L +5V #PWR5
+L +5V #PWR04
 U 1 1 4D51AA08
 P 6350 2900
-F 0 "#PWR5" H 6350 2990 20  0001 C CNN
+F 0 "#PWR04" H 6350 2990 20  0001 C CNN
 F 1 "+5V" H 6350 2990 30  0000 C CNN
 	1    6350 2900
@@
 $EndComp
 $Comp
-L GND #PWR3
+L GND #PWR05
 U 1 1 4D51A9DE
 P 6350 2700
-F 0 "#PWR3" H 6350 2700 30  0001 C CNN
+F 0 "#PWR05" H 6350 2700 30  0001 C CNN
 F 1 "GND" H 6350 2630 30  0001 C CNN
 	1    6350 2700
@@
 $EndComp
 $Comp
-L GND #PWR4
+L GND #PWR06
 U 1 1 4D51A9D5
 P 4150 2900
-F 0 "#PWR4" H 4150 2900 30  0001 C CNN
+F 0 "#PWR06" H 4150 2900 30  0001 C CNN
 F 1 "GND" H 4150 2830 30  0001 C CNN
 	1    4150 2900
@@
 NoConn ~ 7950 2850
 $Comp
-L GND #PWR6
+L GND #PWR07
 U 1 1 4D518B19
 P 8300 3800
-F 0 "#PWR6" H 8300 3800 30  0001 C CNN
+F 0 "#PWR07" H 8300 3800 30  0001 C CNN
 F 1 "GND" H 8300 3730 30  0001 C CNN
 	1    8300 3800
@@
 $EndComp
 $Comp
-L GND #PWR13
+L GND #PWR08
 U 1 1 4AFA0646
 P 3850 5800
-F 0 "#PWR13" H 3850 5800 30  0001 C CNN
+F 0 "#PWR08" H 3850 5800 30  0001 C CNN
 F 1 "GND" H 3850 5730 30  0001 C CNN
 	1    3850 5800
@@
 $EndComp
 $Comp
-L +5V #PWR11
+L +5V #PWR09
 U 1 1 4AFA0642
 P 3850 5300
-F 0 "#PWR11" H 3850 5390 20  0001 C CNN
+F 0 "#PWR09" H 3850 5390 20  0001 C CNN
 F 1 "+5V" H 3850 5390 30  0000 C CNN
 	1    3850 5300
@@
 $EndComp
 $Comp
-L GND #PWR9
+L GND #PWR010
 U 1 1 4AFA063F
 P 3850 5000
-F 0 "#PWR9" H 3850 5000 30  0001 C CNN
+F 0 "#PWR010" H 3850 5000 30  0001 C CNN
 F 1 "GND" H 3850 4930 30  0001 C CNN
 	1    3850 5000
@@
 $EndComp
 $Comp
-L +5V #PWR7
+L +5V #PWR011
 U 1 1 4AFA063C
 P 3850 4500
-F 0 "#PWR7" H 3850 4590 20  0001 C CNN
+F 0 "#PWR011" H 3850 4590 20  0001 C CNN
 F 1 "+5V" H 3850 4590 30  0000 C CNN
 	1    3850 4500
@@
 $EndComp
 $Comp
-L GND #PWR12
-U 1 1 4AF9FB68
-P 5200 5600
-F 0 "#PWR12" H 5200 5600 30  0001 C CNN
-F 1 "GND" H 5200 5530 30  0001 C CNN
-	1    5200 5600
-	1    0    0    -1
-$EndComp
-$Comp
-L +5V #PWR8
-U 1 1 4AF9FB55
-P 5200 4700
-F 0 "#PWR8" H 5200 4790 20  0001 C CNN
-F 1 "+5V" H 5200 4790 30  0000 C CNN
-	1    5200 4700
-	1    0    0    -1
-$EndComp
-$Comp
-L +5V #PWR2
+L +5V #PWR012
 U 1 1 4AF9BF86
 P 6700 2400
-F 0 "#PWR2" H 6700 2490 20  0001 C CNN
+F 0 "#PWR012" H 6700 2490 20  0001 C CNN
 F 1 "+5V" H 6700 2490 30  0000 C CNN
 	1    6700 2400
@@
 $EndComp
 $Comp
-L +5V #PWR1
+L +5V #PWR013
 U 1 1 4AF9BF83
 P 6500 2400
-F 0 "#PWR1" H 6500 2490 20  0001 C CNN
+F 0 "#PWR013" H 6500 2490 20  0001 C CNN
 F 1 "+5V" H 6500 2490 30  0000 C CNN
 	1    6500 2400
